Commit message: fixed another typo

File: description/robot_core.xacro (robot description, xacro)
@@ -90,5 +90,5 @@
     <joint name="caster_wheel_joint" type="fixed">
         <parent link="chassis"/>
-        <chiled link="caster_wheel"/>
+        <child link="caster_wheel"/>
         <origin xyz="0.44 0 0"/>
     </joint>

Commit message: changed robot size

File: description/robot_core.xacro (robot description, xacro)
@@ -25,25 +25,28 @@
     <link name="chassis">
         <visual>
-            <origin xyz="0.25 0 0.1"/>
+            <origin xyz="0.4 0 0.1"/>
             <geometry>
-                <box size="0.5 0.5 0.2"/>
+                <box size="0.8 0.5 0.2"/>
             </geometry>
             <material name="white"/>
         </visual>
         <collision>
-            <origin xyz="0.25 0 0.1"/>
+            <origin xyz="0.4 0 0.1"/>
             <geometry>
-                <box size="0.5 0.5 0.2"/>
+                <box size="0.8 0.5 0.2"/>
             </geometry>
         </collision>
-        <xacro:inertial_box mass="5" x="0.5" y="0.5" z="0.2">
-            <origin xyz="0.25 0 0.1" rpy="0 0 0"/>
+        <xacro:inertial_box mass="5" x="0.8" y="0.5" z="0.2">
+            <origin xyz="0.4 0 0.1" rpy="0 0 0"/>
         </xacro:inertial_box>
     </link>
+    <gazebo reference="chassis">
+        <material>Gazebo/White</material>
+    </gazebo>
     <!-- LEFT WHEEL LINK -->
     <joint name="left_wheel_joint" type="continuous">
         <parent link="base_link"/>
         <child link="left_wheel"/>
-        <origin xyz="0 0.275 0" rpy="-${pi/2} 0 0"/>
+        <origin xyz="0 0.279 0" rpy="-${pi/2} 0 0"/>
         <axis xyz="0 0 1"/>
     </joint>
@@ -51,5 +54,5 @@
         <visual>
             <geometry>
-                <cylinder radius="0.15" length="0.08"/>
+                <cylinder radius="0.1" length="0.07"/>
             </geometry>
             <material name="black"/>
@@ -57,16 +60,19 @@
         <collision>
             <geometry>
-                <cylinder radius="0.15" length="0.08"/>
+                <cylinder radius="0.1" length="0.07"/>
             </geometry>
         </collision>
-        <xacro:inertial_cylinder mass="0.1" length="0.08" radius="0.15">
+        <xacro:inertial_cylinder mass="0.1" length="0.07" radius="0.1">
             <origin xyz="0 0 0" rpy="0 0 0"/>
         </xacro:inertial_cylinder>
     </link>
+    <gazebo reference="left_wheel">
+        <material>Gazebo/Black</material>
+    </gazebo>
     <!-- RIGHT WHEEL LINK -->
     <joint name="right_wheel_joint" type="continuous">
         <parent link="base_link"/>
         <child link="right_wheel"/>
-        <origin xyz="0 -0.275 0" rpy="${pi/2} 0 0"/>
+        <origin xyz="0 -0.279 0" rpy="${pi/2} 0 0"/>
         <axis xyz="0 0 -1"/>
     </joint>
@@ -74,5 +80,5 @@
         <visual>
             <geometry>
-                <cylinder radius="0.15" length="0.08"/>
+                <cylinder radius="0.1" length="0.07"/>
             </geometry>
             <material name="black"/>
@@ -80,21 +86,24 @@
         <collision>
             <geometry>
-                <cylinder radius="0.15" length="0.08"/>
+                <cylinder radius="0.1" length="0.07"/>
             </geometry>
         </collision>
-        <xacro:inertial_cylinder mass="0.1" length="0.08" radius="0.15">
+        <xacro:inertial_cylinder mass="0.1" length="0.07" radius="0.1">
             <origin xyz="0 0 0" rpy="0 0 0"/>
         </xacro:inertial_cylinder>
     </link>
+    <gazebo reference="right_wheel">
+        <material>Gazebo/Black</material>
+    </gazebo>
     <!-- CASTER WHEEL LINK-->
     <joint name="caster_wheel_joint" type="fixed">
         <parent link="chassis"/>
         <child link="caster_wheel"/>
-        <origin xyz="0.44 0 0"/>
+        <origin xyz="0.6 0 0"/>
     </joint>
         <link name ="caster_wheel">
         <visual>
             <geometry>
-                <sphere radius="0.15"/>
+                <sphere radius="0.1"/>
             </geometry>
             <material name="black"/>
@@ -102,10 +111,13 @@
         <collision>
             <geometry>
-                <sphere radius="0.15"/>
+                <sphere radius="0.1"/>
             </geometry>
         </collision>
-        <xacro:inertial_sphere mass="0.1" radius="0.15">
+        <xacro:inertial_sphere mass="0.1" radius="0.1">
             <origin xyz="0 0 0" rpy="0 0 0"/>
         </xacro:inertial_sphere>
     </link>
+    <gazebo reference="caster_wheel">
+        <material>Gazebo/Black</material>
+    </gazebo>
 </robot>

Commit message: Updated Robot size

File: description/robot_core.xacro (robot description, xacro)
@@ -36,18 +36,18 @@
     <link name="chassis">
         <visual>
-            <origin xyz="0.4 0 0.1"/>
+            <origin xyz="0.25 0 0.1"/>
             <geometry>
-                <box size="0.8 0.5 0.2"/>
+                <box size="0.5 0.5 0.2"/>
             </geometry>
             <material name="white"/>
         </visual>
         <collision>
-            <origin xyz="0.4 0 0.1"/>
+            <origin xyz="0.25 0 0.1"/>
             <geometry>
-                <box size="0.8 0.5 0.2"/>
+                <box size="0.5 0.5 0.2"/>
             </geometry>
         </collision>
-        <xacro:inertial_box mass="5" x="0.8" y="0.5" z="0.2">
-            <origin xyz="0.4 0 0.1" rpy="0 0 0"/>
+        <xacro:inertial_box mass="5" x="0.5" y="0.5" z="0.2">
+            <origin xyz="0.25 0 0.1" rpy="0 0 0"/>
         </xacro:inertial_box>
     </link>
@@ -111,5 +111,5 @@
         <parent link="chassis"/>
         <child link="caster_wheel"/>
-        <origin xyz="0.6 0 0"/>
+        <origin xyz="0.4 0 0"/>
     </joint>
         <link name ="caster_wheel">
